File: ESC_Board/ESC_Board.kicad_sch (KiCad schematic)
At the start: 69 parts, among them Q1 SIR182DP-T1-RE3, Q2 SIR182DP-T1-RE3, Q3 SIR182DP, Q4 SIR182DP, Q5 SIR182DP, Q6 SIR182Dp, Q7 SIR182DP, Q8 SIR182DP, U1 INA180A3, U2 STM32F051K8Ux, U3 IR2104, U4 TPS62153RGTT, U5 DRV8300DRGER, U6 TLV76601QWDRBRQ1, U7 INA180A3

Commit message: ESC Board: Finalized ESC design
Parts:
- removed C1, C2: 1uF, PCM_JLCPCB:C_0603, symbol PCM_JLCPCB-Capacitors:0603,1uF
- removed C14: 1uF, PCM_JLCPCB:C_0402, symbol PCM_JLCPCB-Capacitors:0402,1uF
- removed C17, C18, C19, C22, C4: 100nF, PCM_JLCPCB:C_0402, symbol PCM_JLCPCB-Capacitors:0402,100nF,(2)
- removed C3: 47u, symbol Device:C
- removed C5: 1nF, PCM_JLCPCB:C_0402, symbol PCM_JLCPCB-Capacitors:0402,1nF
- removed C6: 10nF, PCM_JLCPCB:C_0603, symbol PCM_JLCPCB-Capacitors:0603,10nF
- removed D1: D_Zener, symbol Device:D_Zener
- removed D2: D_Small, symbol Device:D_Small
- removed Q1, Q2: SIR182DP-T1-RE3, Package_TO_SOT_SMD:TDSON-8-1, symbol Transistor_FET:BSC13DN30NSFD
- removed R1, R6: 1kΩ, PCM_JLCPCB:R_0402, symbol PCM_JLCPCB-Resistors:0402,1kΩ
- removed R12, R5: 2m, symbol Device:R_Small
- removed R15, R16, R17, R18, R19, R2, R20, R3: 100Ω, PCM_JLCPCB:R_0603, symbol PCM_JLCPCB-Resistors:0603,100Ω
- removed R4: 4.7kΩ, PCM_JLCPCB:R_0402, symbol PCM_JLCPCB-Resistors:0402,4.7kΩ
- removed U1, U7: INA180A3, Package_TO_SOT_SMD:SOT-23-5, symbol Amplifier_Current:INA180A3
- removed U3: IR2104, symbol Driver_FET:IR2104
- added C1: 100nF, PCM_JLCPCB:C_0402, symbol PCM_JLCPCB-Capacitors:0402,100nF,(2)
- added C23, C24, C25, C26, C52: 1uF, PCM_JLCPCB:C_0603, symbol PCM_JLCPCB-Capacitors:0603,1uF
- added C5: 100uF, Capacitor_SMD:CP_Elec_8x10, symbol Device:C_Polarized_Small
- added D1: Red, PCM_JLCPCB:D_0805, symbol PCM_JLCPCB-Diodes:LED,0805,Red
- added D8: SMBJ18A, PCM_JLCPCB:D_SMB, symbol PCM_JLCPCB-Diodes:TVS-Uni,SMBJ18A
- added Q1: AO3400A, PCM_JLCPCB:Q_SOT-23, symbol PCM_JLCPCB-Transistors:NMOS,AO3400A
- added R1: R_Shunt, symbol Device:R_Shunt
- added R12: 10kΩ, PCM_JLCPCB:R_0402, symbol PCM_JLCPCB-Resistors:0402,10kΩ
- added R15, R16, R17, R18, R19, R20: 22Ω, PCM_JLCPCB:R_0402, symbol PCM_JLCPCB-Resistors:0402,22Ω
- added R2: 1kΩ, PCM_JLCPCB:R_0603, symbol PCM_JLCPCB-Resistors:0603,1kΩ
- added R3: 75Ω, PCM_JLCPCB:R_0603, symbol PCM_JLCPCB-Resistors:0603,75Ω
- added TP2: TestPoint_2Pole, symbol Connector:TestPoint_2Pole
- added U3: INA180A1, Package_TO_SOT_SMD:SOT-23-5, symbol Amplifier_Current:INA180A1
- C20: LCSC C15849 -> C6119857; Manufacturer Samsung Electro-Mechanics -> (none); Part CL10A105KB8NNNC -> (none)
Connections:
- net SHA is gone; now on net MOTORA: Q3.5 (D), Q5.1 (S), Q5.2 (S), Q5.3 (S), U5.18 (SHA)
- net SHB is gone; now on net MOTORB: Q4.5 (D), Q6.1 (S), Q6.2 (S), Q6.3 (S), U5.15 (SHB)
- net SHC is gone; now on net MOTORC: Q7.1 (S), Q7.2 (S), Q7.3 (S), Q8.5 (D), U5.12 (SHC)
- net +17V: now also C5.1, C52.1, D8.2
- net +3.3V: now also C26.1, D1.2, U3.5 (V+)
- net BEMFA: now also U2.7 (PA1)
- net BEMFB: now also U2.8 (PA2)
- net BEMFC: now also U2.9 (PA3)
- net BEMFCOMMON: now also U2.6 (PA0)
- net GHA: now also R15.1
- net GHB: now also R17.1
- net GHC: now also R19.1
- net GLA: now also R16.1
- net GLB: now also R18.1, R20.1
- net GND: now also C1.2, C26.2, C5.2, C52.2, Q1.2 (S), R1.4, R12.1, U3.2 (GND); no longer Q3.1 (S), Q3.2 (S), Q3.3 (S), Q4.1 (S), Q4.2 (S), Q4.3 (S), Q8.1 (S), Q8.2 (S), Q8.3 (S)
- net MOTORA: now also C23.2
- net MOTORB: now also C24.2
- net MOTORC: now also C25.2
- net SWDR: now also TP2.2
- net UART2_RX: now also U2.30 (PB7); no longer U2.9 (PA3)
- net UART2_TX: now also U2.29 (PB6); no longer U2.8 (PA2)
- net at Q4.4 (G): now also R18.2
- net at Q8.4 (G): now also R20.2
- net at Q6.4 (G): now also R17.2
- net at Q5.4 (G): now also R15.2
- net INLA: now reaches U5.1 (INLA)
- net INLA: now also U2.13 (PA7)
- net at U5.14 (BSTC): now also C25.1
- net at U5.17 (BSTB): now also C24.1
- net INLB: now reaches U5.2 (INLB)
- net INLB: now also U2.14 (PB0)
- net at U5.20 (BSTA): now also C23.1
- net INHA: now reaches U5.22 (INHA)
- net INHA: now also U2.18 (PA8)
- net INHB: now reaches U5.23 (INHB)
- net INHB: now also U2.19 (PA9)
- net INHC: now reaches U5.24 (INHC)
- net INHC: now also U2.20 (PA10)
- net INCA: now reaches U5.3 (INLC)
- net at Q7.4 (G): now also R19.2
- net at Q3.4 (G): now also R16.2
- net I_SENSE: now reaches U2.10 (PA4)
- net I_SENSE: now also C1.1, R2.2
- net INLC: now reaches U2.15 (PB1)
- net at U2.32 (PB8): now also Q1.1 (G)
- new net: D1.1, R3.2
- new net: R12.2, TP2.1
- new net: Q1.3 (D), R3.1
- new net: R2.1, U3.1
- new net: R1.2, U3.3 (+)
- new net: R1.3, U3.4 (-)
- new net -LiPo: D8.1
- new net LOW_COMMON: Q3.1 (S), Q3.2 (S), Q3.3 (S), Q4.1 (S), Q4.2 (S), Q4.3 (S), Q8.1 (S), Q8.2 (S), Q8.3 (S), R1.1
- no-connect marks 7 -> 14
Other:
- added sheet ESC2.sch (ESC1.kicad_sch)
- added sheet ESC3.sch1 (ESC1.kicad_sch)
- added sheet ESC4.sch2 (ESC1.kicad_sch)
- note added: "BEMF Circuit"
- note added: "CURRENT SENSE"
- note added: "LDO"
- note added: "TIM_CH1"
- note added: "TIM_CH1N"
- note added: "TIM_CH2"
- note added: "TIM_CH2N"
- note added: "TIM_CH3"
- note added: "TIM_CH3N"
- note added: "TVS"
- note added: "low gain as to not overwhelm pin"
- note removed: "100 V/V gain"
- note removed: "look into sizing for power disipation, look into choosing decoupling capacitors, H bridges, etc"
- note removed: "shunt resistor to measure current"
- note removed: "spec out PWR dissipitation"
- note removed: "steps down voltage thus MCU can handle it"
- moved on the sheet: C10, C12, C15, C16, C20, C21, C7, C9, D3, Q3, Q4, Q5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
