File: ESC_Board/ESC1.kicad_sch (KiCad schematic)
At the start: 47 parts, among them Q10 SIR182DP, Q11 SIR182Dp, Q12 SIR182DP, Q13 SIR182DP, Q14 SIR182DP, Q2 AO3400A, Q9 SIR182DP, U7 STM32F051K8Ux, U8 DRV8300DRGER, U9 INA180A1

Commit message: Began PCB design
Parts:
- removed R5: R_Shunt, symbol Device:R_Shunt
- added R95: 3.0m, Resistor_SMD:R_2512_6332Metric, symbol Device:R_Small
- R28, R29, R30: LCSC C25744 -> C191123; Manufacturer UNI-ROYAL(Uniroyal Elec) -> (none); Operating Temperature Range -55°C~+155°C -> (none); Overload Voltage (Max) 50V -> (none); Part 0402WGF1002TCE -> (none); Power(Watts) 62.5mW -> 100mW
- R31, R32, R33, R34, R38, R39, R45, R46: LCSC C25092 -> C400511; Manufacturer UNI-ROYAL(Uniroyal Elec) -> (none); Operating Temperature Range -55°C~+155°C -> (none); Overload Voltage (Max) 50V -> (none); Part 0402WGF220JTCE -> (none); Power(Watts) 62.5mW -> 100mW
- R35, R37, R40, R42, R43, R47: footprint PCM_JLCPCB:R_0603 -> PCM_JLCPCB:R_0402; LCSC C25804 -> C191123; Manufacturer UNI-ROYAL(Uniroyal Elec) -> (none); Operating Temperature Range -55°C~+155°C -> (none); Overload Voltage (Max) 75V -> (none); Part 0603WAF1002T5E -> (none)
- R36, R41, R44, R6: footprint PCM_JLCPCB:R_0603 -> PCM_JLCPCB:R_0402; LCSC C21190 -> C2759467; Manufacturer UNI-ROYAL(Uniroyal Elec) -> (none); Operating Temperature Range -55°C~+155°C -> (none); Overload Voltage (Max) 75V -> (none); Part 0603WAF1001T5E -> HP02WAJ0102TCE
- R4: footprint PCM_JLCPCB:R_0603 -> PCM_JLCPCB:R_0402; Manufacturer UNI-ROYAL(Uniroyal Elec) -> (none); Operating Temperature Range -55°C~+155°C -> (none); Overload Voltage (Max) 75V -> (none); Part 0603WAF750JT5E -> 0402WGF750JTCE; Power(Watts) 100mW -> 62.5mW
Connections:
- net INCA is gone; now on net INLC: U8.3 (INLC)
- net GLB: no longer R46.1, U8.9 (GLC)
- net GND: now also U9.4 (-), R95.2
- net LOW_COMMON: now also U9.3 (+), R95.1
- new net GLC: R46.1, U8.9 (GLC)
