File: ESC_Board/ESC_Board.kicad_pcb (KiCad board)
At the start: 4 copper layers, 57.4 x 50.8 mm, 193 parts, among them Q1 AO3400A, Q10 SIR182DP, Q11 SIR182Dp, Q12 SIR182DP, Q13 SIR182DP, Q14 SIR182DP, Q15 AO3400A, Q16 SIR182DP, Q17 SIR182DP, Q18 SIR182Dp, Q19 SIR182DP, Q2 AO3400A, Q20 SIR182DP, Q21 SIR182DP, Q22 AO3400A, Q23 SIR182DP, Q24 SIR182DP, Q25 SIR182Dp, Q26 SIR182DP, Q27 SIR182DP, Q28 SIR182DP, Q3 SIR182DP, Q4 SIR182DP, Q5 SIR182DP, Q6 SIR182Dp, Q7 SIR182DP, Q8 SIR182DP, Q9 SIR182DP, U10 DRV8300DRGER, U11 STM32F051K8Ux, U12 INA180A1, U13 DRV8300DRGER, U14 STM32F051K8Ux, U15 INA180A1, U2 STM32F051K8Ux, U3 INA180A1, U4 TPS62153RGTT, U5 DRV8300DRGER, U6 TLV76601QWDRBRQ1, U7 STM32F051K8Ux, U8 DRV8300DRGER, U9 INA180A1

Commit message: DroneController: Adjusted crystal oscillator, added SWD debugging
Parts:
- added C6: 100uF, Capacitor_SMD:CP_Elec_8x10, F.Cu at (56.8, 139.2)
- added J1: 63824-1, footprints:TRM2_63824-1_TEC, F.Cu at (99.1, 94.7)
- added J2: 63824-1, footprints:TRM2_63824-1_TEC, F.Cu at (107.8, 109.5)
- added J3: 63824-1, footprints:TRM2_63824-1_TEC, F.Cu at (107.6, 124.2)
- added Q3: SIR182DP, Package_TO_SOT_SMD:TDSON-8-1, F.Cu at (58.4, 86.3)
- added Q5: SIR182DP, Package_TO_SOT_SMD:TDSON-8-1, F.Cu at (58.4, 80.2)
- moved U4 38.7 mm to (87.7, 135.0)
- moved C11 38.7 mm to (90.5, 133.5)
- moved C13 38.7 mm to (90.5, 136.6)
- moved C53 38.7 mm to (86.3, 131.0)
- moved C54 38.7 mm to (86.3, 132.3)
- moved L1 38.7 mm to (83.5, 133.8)
- moved R7 38.7 mm to (84.6, 137.1)
- moved R27 25.0 mm to (55.6, 124.6)
- moved R22 22.1 mm to (52.1, 108.3)
- moved R23 22.1 mm to (52.1, 109.2)
- moved Q8 20.3 mm to (102.8, 121.0)
- moved R18 19.8 mm to (99.5, 103.5)
- moved R20 19.7 mm to (99.0, 118.1), turned to 0 degrees
- moved Q4 19.7 mm to (102.8, 106.3)
- moved R26 18.3 mm to (55.5, 117.0)
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Connections:
- U4 pad 6: GND -> AGND
Routing:
- net /LOW_COMMON: track 1.47 -> 48.3 mm, vias 1 -> 4
- net /GLB: track 1.21 -> 16.1 mm, vias 1 -> 2
- net /GHC: track 2.04 -> 16.8 mm, vias 1 -> 2
- net /GLA: track 1.09 -> 13.0 mm, vias 1 -> 2
- net /GLC: track 1.57 -> 11.5 mm, vias 1 -> 2
- net /GHA: track 16.6 -> 6.68 mm
- net /GHB: track 2.07 -> 5.72 mm, vias 1 -> 2
- net Net-(Q3-G): track 0.00 -> 2.91 mm
- net /MOTORA: track 2.54 -> 0.00 mm, vias 2 -> 0
- net Net-(Q4-G): track 0.00 -> 1.59 mm
- net Net-(Q7-G): track 0.00 -> 1.32 mm
- net /INLA: track 2.93 -> 3.90 mm
- net /MOTORB: track 1.32 -> 2.01 mm, vias 3 -> 0
- net /MOTORC: track 2.41 -> 2.66 mm, vias 2 -> 0
- net (no net): vias 2 -> 0
- added copper zone on In2.Cu, net +17V
Other:
- board size 57.4 x 50.8 mm -> 73.2 x 50.8 mm
